File: PCB/tarocco.brd (EAGLE design)
At the start: 40 x 40 mm, 42 parts, among them IC1 CY8C4545PVI, Q1 NEXFET_SINGLECSD18537NQ5A, Q2 NEXFET_SINGLECSD18537NQ5A, Q3 NEXFET_SINGLECSD18537NQ5A, Q4 NEXFET_SINGLECSD18537NQ5A

Commit message: Initial Commit of Schematic
Parts:
- added C12, C13, C14: 0.1uF, SparkFun-Capacitors:0603
- added C15: 100uF, SparkFun-Capacitors:CPOL-RADIAL-2.5MM-6.5MM
- added C16: 1nF, SparkFun-Capacitors:0603
- added J1, J2: (no value), SparkFun-Connectors:1X02_LONGPADS
- added MOTOR, SUPPLY: JST-XH-02-PIN-LONG-PAD, JST XH Connectors v1-0:JST-XH-02-PACKAGE-LONG-PAD
- added R13, R14: 10k, SparkFun-Resistors:0603
- added R15: 100k, SparkFun-Resistors:0603
- added R16: .2, SparkFun-Resistors:2010
- added U1: DRV8801PWP, DRV8801PWP:SOP65P640X120-17N
- MTR, PSU: device SparkFun-Connectors:SCREWTERMINAL-3.5MM-2 -> SparkFun-Connectors:SCREWTERMINAL-3.5MM-2@1
Connections:
- new net N$26: C13.1, C14.2, C15.1, J2.1, SUPPLY.1, U1.9
- new net N$27: R15.1, U1.15
- new net N$28: C12.1, U1.11
- new net N$30: C12.2, U1.12
- new net N$31: C13.2, U1.14
- new net N$32: R14.2, U1.16
- new net N$36: R16.2, U1.8
- new net N$37: J1.1, MOTOR.1, U1.7
- new net N$38: J1.2, MOTOR.2, U1.10
- new net N$9: R13.2, U1.2
- net 5V: now also R13.1
- net ENABLE: now also U1.6
- net FAULT: now also U1.1
- net GND: now also C14.1, C15.2, C16.2, J2.2, R14.1, R16.1, SUPPLY.2, U1.13, U1.17, U1.4
- net ISENSE: now also C16.1, R15.2
- net PHASE: now also U1.3
- net SLEEP: now also U1.5

Commit message: Time to sleep, routing is hard
Parts:
- removed 8701: DRV8701, drv8x:VQFN24
- removed C10, C9: (no value), adafruit:E3,5-8
- removed C4, C7, C8: 1u, adafruit:C0603
- removed C5, C6: 100n, adafruit:C0603
- removed MTR, PSU: M023.5MM, SparkFun-Connectors:SCREWTERMINAL-3.5MM-2@1
- removed Q1, Q2, Q3, Q4: NEXFET_SINGLECSD18537NQ5A, mosfet:SON5X6
- removed R3, R4: 1k, adafruit:R0603
- removed R5: 200k, adafruit:R0603
- removed R6: 68k, adafruit:R0603
- removed RSENSE: 0.005, adafruit:R2512
- R16: value .2 -> 0.1; device SparkFun-Resistors:2010 -> SparkFun-Resistors:1210
- moved J2 128.5 mm to (12.7, 1.27), turned to 90 degrees
- moved J1 127.6 mm to (21.6, 17.8), turned to 180 degrees
- moved MOTOR 115.5 mm to (20.3, 23.5), turned to 180 degrees
- moved R16 101.0 mm to (25.4, 17.8), turned to 270 degrees
- moved C16 95.5 mm to (29.2, 10.2), turned to 270 degrees
- moved R13 88.1 mm to (31.1, 13.3), turned to 180 degrees
- moved R15 86.8 mm to (21.6, 7.62)
- moved R14 83.0 mm to (19.7, 8.26), turned to 180 degrees
- moved STANDOFF4 80.6 mm to (-44.5, 31.8)
- moved C15 66.6 mm to (29.2, 3.81), turned to 180 degrees
- moved STANDOFF2 62.9 mm to (-31.8, 31.8)
- moved C14 58.7 mm to (16.5, 7.62), turned to 180 degrees
- moved C13 54.4 mm to (11.4, 8.89), turned to 90 degrees
- moved C12 53.8 mm to (12.1, 12.1), turned to 270 degrees
- moved STANDOFF3 50.3 mm to (-38.1, 31.8)
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Connections:
- net N$37 renamed VMOT+
- net N$38 renamed VMOT-
- removed net N$1: 8701.GL1, Q3.GATE
- removed net N$11: 8701.VCP, C4.2
- removed net N$12: 8701.CPL, C5.2
- removed net N$13: 8701.CPH, C5.1
- removed net N$15: 8701.VREF, R3.1, R4.1
- removed net N$16: 8701.AVDD, C7.1, R4.2, R6.1
- removed net N$17: 8701.DVDD, C8.1
- removed net N$2: 8701.SH1, MTR.2, Q3.DRAIN@1, Q3.DRAIN@2, Q3.DRAIN@3, Q3.DRAIN@4, Q3.DRAIN@5, Q4.SOURCE@1, Q4.SOURCE@2, Q4.SOURCE@3
- removed net N$21: 8701.IDRIVE, R5.2, R6.2
- removed net N$23: 8701.VM, C10.+, C4.1, C6.1, C9.+, PSU.1, Q1.DRAIN@1, Q1.DRAIN@2, Q1.DRAIN@3, Q1.DRAIN@4, Q1.DRAIN@5, Q4.DRAIN@1, Q4.DRAIN@2, Q4.DRAIN@3, Q4.DRAIN@4, Q4.DRAIN@5
- removed net N$3: 8701.SH2, MTR.1, Q1.SOURCE@1, Q1.SOURCE@2, Q1.SOURCE@3, Q2.DRAIN@1, Q2.DRAIN@2, Q2.DRAIN@3, Q2.DRAIN@4, Q2.DRAIN@5
- removed net N$4: 8701.GH2, Q1.GATE
- removed net N$5: 8701.SP, Q2.SOURCE@1, Q2.SOURCE@2, Q2.SOURCE@3, Q3.SOURCE@1, Q3.SOURCE@2, Q3.SOURCE@3, RSENSE.2
- removed net N$6: 8701.GL2, Q2.GATE
- removed net N$7: 8701.GH1, Q4.GATE
- net ENABLE: no longer 8701.EN
- net FAULT: no longer 8701.FAULT
- net GND: no longer 8701.GND@1, 8701.GND@2, 8701.GND@3, 8701.SN, C10.-, C6.2, C7.2, C8.2, C9.-, PSU.2, R3.2, R5.1, RSENSE.1
- net ISENSE: no longer 8701.SO
- net OVC: no longer 8701.SENSE
- net PHASE: no longer 8701.PH
- net SLEEP: no longer 8701.SLEEP
Routing:
- net 5V: track 57.0 -> 0.00 mm, vias 1 -> 0
- net N$2: track 24.7 -> 0.00 mm, vias 2 -> 0
- net RXD: track 22.6 -> 0.00 mm
- net TXD: track 20.3 -> 0.00 mm
- net N$7: track 19.9 -> 0.00 mm
- net N$4: track 18.2 -> 0.00 mm, vias 2 -> 0
- net XRES: track 17.2 -> 0.00 mm, vias 1 -> 0
- net SWDIO: track 16.1 -> 0.00 mm, vias 1 -> 0
- net FAULT: track 15.1 -> 0.00 mm
- net SWDCLK: track 14.9 -> 0.00 mm, vias 1 -> 0
- net OVC: track 14.3 -> 0.00 mm
- net DIRECTION: track 13.8 -> 0.00 mm
- net ISENSE: track 13.5 -> 0.00 mm
- net N$1: track 13.4 -> 0.00 mm
- net N$6: track 13.0 -> 0.00 mm
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- added copper zone on layer 1, net VMOT+
- added copper zone on layer 1, net VMOT-
- removed copper zone on layer 1, net GND
- removed copper zone on layer 1, net N$2
- removed copper zone on layer 1, net N$23
- removed copper zone on layer 16, net N$23
- removed copper zone on layer 1, net N$3
- removed copper zone on layer 1, net N$5
Other:
- board size 40 x 40 mm -> 47 x 26.3 mm
- board text removed: "27.5"
- board text removed: "3.5"
- board text removed: "33"
- board text removed: "40"
- board text removed: "5V"
- board text removed: "A"
- board text removed: "All dimensions in mm"
- board text removed: "B"
- board text removed: "CITRUS CNC"
- board text removed: "DIR"
- board text removed: "DIRECTION"
- board text removed: "ERR"
- board text removed: "ERROR"
- board text removed: "GND"
- board text removed: "MOTOR-A"
- board text removed: "MOTOR-B"
- board text removed: "RES"
- board text removed: "RESET"
- board text removed: "RXD"
- board text removed: "STEP"
- board text removed: "STP"
- board text removed: "TXD"
- board text removed: "V+"
- board text removed: "V-"
- board text removed: "VLOGIC"
