File: PCB/Tarocco-Lite.sch (EAGLE design)
At the start: 37 parts, among them IC1 CY8C4545PVI, U1 DRV8801PWP

Commit message: Rename and mostly routed
Parts:
- removed J1, J2: (no value), SparkFun-Connectors:CONN_02PTH3
Connections:
- net N$36 renamed SENSE
- removed net N$26: C13.1, C14.2, C15.+, J2.1, SUPPLY-1.S, U1.VBB
- new net VBB: C13.1, C14.2, C15.+, SUPPLY-1.S, U1.VBB
- net GND: no longer J2.2
- net VMOT+: no longer J1.1
- net VMOT-: no longer J1.2
Changed lines of the file:
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@@
 <part name="R16" library="SparkFun-Resistors" deviceset="0.1OHM" device="-1210-1/2W-1%" value="0.1"/>
 <part name="MOTOR" library="JST XH Connectors v1-0" deviceset="JST-XH-02-PIN" device="-LONG-PAD"/>
-<part name="J1" library="SparkFun-Connectors" deviceset="CONN_02" device="PTH3"/>
-<part name="J2" library="SparkFun-Connectors" deviceset="CONN_02" device="PTH3"/>
-<part name="GND16" library="SparkFun-Aesthetics" deviceset="GND" device=""/>
 </parts>
 <sheets>
@@
 <instance part="MOTOR" gate="-2" x="246.38" y="93.98"/>
 <instance part="MOTOR" gate="-1" x="246.38" y="96.52"/>
-<instance part="J1" gate="G$1" x="238.76" y="106.68" rot="R270"/>
-<instance part="J2" gate="G$1" x="175.26" y="109.22" rot="R270"/>
-<instance part="GND16" gate="1" x="177.8" y="99.06"/>
 </instances>
 <busses>
@@
 <wire x1="266.7" y1="66.04" x2="266.7" y2="73.66" width="0.1524" layer="91"/>
 </segment>
-<segment>
-<pinref part="J2" gate="G$1" pin="2"/>
-<pinref part="GND16" gate="1" pin="GND"/>
-</segment>
 </net>
 <net name="5V" class="0">
@@
 </segment>
 </net>
-<net name="N$26" class="0">
+<net name="VBB" class="0">
 <segment>
 <pinref part="SUPPLY" gate="-1" pin="S"/>
@@
 <pinref part="C13" gate="G$1" pin="1"/>
 <wire x1="149.86" y1="96.52" x2="165.1" y2="96.52" width="0.1524" layer="91"/>
-<wire x1="165.1" y1="96.52" x2="175.26" y2="96.52" width="0.1524" layer="91"/>
-<wire x1="175.26" y1="96.52" x2="198.12" y2="96.52" width="0.1524" layer="91"/>
+<wire x1="165.1" y1="96.52" x2="198.12" y2="96.52" width="0.1524" layer="91"/>
 <wire x1="149.86" y1="86.36" x2="149.86" y2="96.52" width="0.1524" layer="91"/>
 <junction x="149.86" y="96.52"/>
@@
 <wire x1="165.1" y1="109.22" x2="165.1" y2="99.06" width="0.1524" layer="91"/>
 <junction x="165.1" y="99.06"/>
-<pinref part="J2" gate="G$1" pin="1"/>
-<wire x1="175.26" y1="96.52" x2="175.26" y2="101.6" width="0.1524" layer="91"/>
-<junction x="175.26" y="96.52"/>
 </segment>
 </net>
@@
 </segment>
 </net>
-<net name="N$36" class="0">
+<net name="SENSE" class="0">
 <segment>
 <pinref part="U1" gate="A" pin="SENSE"/>
@@
 <pinref part="MOTOR" gate="-1" pin="S"/>
 <pinref part="U1" gate="A" pin="OUT+"/>
-<wire x1="243.84" y1="96.52" x2="238.76" y2="96.52" width="0.1524" layer="91"/>
-<pinref part="J1" gate="G$1" pin="1"/>
-<wire x1="238.76" y1="96.52" x2="233.68" y2="96.52" width="0.1524" layer="91"/>
-<wire x1="238.76" y1="99.06" x2="238.76" y2="96.52" width="0.1524" layer="91"/>
-<junction x="238.76" y="96.52"/>
+<wire x1="243.84" y1="96.52" x2="233.68" y2="96.52" width="0.1524" layer="91"/>
 </segment>
 </net>
@@
 <pinref part="MOTOR" gate="-2" pin="S"/>
 <pinref part="U1" gate="A" pin="OUT-"/>
-<wire x1="243.84" y1="93.98" x2="241.3" y2="93.98" width="0.1524" layer="91"/>
-<pinref part="J1" gate="G$1" pin="2"/>
-<wire x1="241.3" y1="93.98" x2="233.68" y2="93.98" width="0.1524" layer="91"/>
-<wire x1="241.3" y1="99.06" x2="241.3" y2="93.98" width="0.1524" layer="91"/>
-<junction x="241.3" y="93.98"/>
-</segment>
-</net>
+<wire x1="243.84" y1="93.98" x2="233.68" y2="93.98" width="0.1524" layer="91"/>
+</segment>
+</net>

Commit message: Alpha finished
Parts:
- removed STANDOFF1, STANDOFF2, STANDOFF3, STANDOFF4: STAND-OFF, SparkFun-Electromechanical:STAND-OFF
Changed lines of the file:
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@@
 <parts>
 <part name="CONTROL" library="jst-ph" deviceset="JST-PH6" device=""/>
-<part name="STANDOFF1" library="SparkFun-Electromechanical" deviceset="STAND-OFF" device=""/>
-<part name="STANDOFF2" library="SparkFun-Electromechanical" deviceset="STAND-OFF" device=""/>
-<part name="STANDOFF3" library="SparkFun-Electromechanical" deviceset="STAND-OFF" device=""/>
-<part name="STANDOFF4" library="SparkFun-Electromechanical" deviceset="STAND-OFF" device=""/>
 <part name="ENCODER" library="jst-ph" deviceset="JST-PH4" device=""/>
 <part name="C2" library="adafruit" deviceset="C-US" device="C0603" value="1u"/>
@@
 <instances>
 <instance part="CONTROL" gate="A" x="15.24" y="124.46"/>
-<instance part="STANDOFF1" gate="G$1" x="5.08" y="129.54"/>
-<instance part="STANDOFF2" gate="G$1" x="5.08" y="114.3"/>
-<instance part="STANDOFF3" gate="G$1" x="5.08" y="124.46"/>
-<instance part="STANDOFF4" gate="G$1" x="5.08" y="119.38"/>
 <instance part="ENCODER" gate="A" x="68.58" y="121.92"/>
 <instance part="C2" gate="G$1" x="106.68" y="91.44" smashed="yes">

Commit message: BOM and labelling update
Parts:
- R16: value 0.1 -> 0.2
Changed lines of the file:
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@@
 <part name="C16" library="SparkFun-Capacitors" deviceset="1.0NF/1000PF" device="-0603-50V-10%" value="1nF"/>
 <part name="GND15" library="SparkFun-Aesthetics" deviceset="GND" device=""/>
-<part name="R16" library="SparkFun-Resistors" deviceset="0.1OHM" device="-1210-1/2W-1%" value="0.1"/>
+<part name="R16" library="SparkFun-Resistors" deviceset="0.1OHM" device="-1210-1/2W-1%" value="0.2"/>
 <part name="MOTOR" library="JST XH Connectors v1-0" deviceset="JST-XH-02-PIN" device="-LONG-PAD"/>
 </parts>

Commit message: SO MUCH CLEANER
Cleaned up a lot of the layout to reduce crosstalk
Parts:
- C15: device SparkFun-Capacitors:100UF-POLAR-RADIAL-2.5MM-25V-20% -> SparkFun-Capacitors:100UF-POLAR-25V-20%(ELEC)
Changed lines of the file:
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@@
 <part name="C13" library="SparkFun-Capacitors" deviceset="0.1UF" device="-0603-25V-(+80/-20%)" value="0.1uF"/>
 <part name="C14" library="SparkFun-Capacitors" deviceset="0.1UF" device="-0603-25V-(+80/-20%)" value="0.1uF"/>
-<part name="C15" library="SparkFun-Capacitors" deviceset="100UF-POLAR" device="-RADIAL-2.5MM-25V-20%" value="100uF"/>
+<part name="C15" library="SparkFun-Capacitors" deviceset="100UF-POLAR" device="-25V-20%(ELEC)" value="100uF"/>
 <part name="R13" library="SparkFun-Resistors" deviceset="10KOHM" device="-0603-1/10W-1%" value="10k"/>
 <part name="R14" library="SparkFun-Resistors" deviceset="10KOHM" device="-0603-1/10W-1%" value="10k"/>
@@
 </sheet>
 </sheets>
+<errors>
+</errors>
 </schematic>
 </drawing>
